Commit message: description: fix xacro wheel macro
Signed-off-by: jean.laneurit <jean.laneurit@inrae.fr>

File: cinteo_description/urdf/visual/wheels.xacro (robot description, xacro)
@@ -22,5 +22,5 @@
         <xacro:rear_wheel_visual />
     </xacro:macro>
-    <xacro:macro name="front_wheel_visual" params="orientation">
+    <xacro:macro name="front_wheel_visual">
         <xacro:wheel_visual
             mesh_filename="package://cinteo_description/meshes/front_wheel.stl" />
