Commit message: [description] update ros2_control xacro file
Signed-off-by: Jean Laneurit <jean.laneurit@inrae.fr>

File: cinteo_description/ros2_control/cinteo.ros2_control.xacro (robot description, xacro)
@@ -45,10 +45,27 @@
     <xacro:property name="maximal_wheel_speed"
       value="${props['rear_wheels_speed_control']['command']['maximal_speed']}" />
-    <!-- hardware plugins -->
-    <xacro:property name="simulation_hardware_plugin"
-      value="romea_mobile_base_gazebo/GazeboSystemInterface1FAS2RWD" />
-    <xacro:property name="live_hardware_plugin"
-      value="cinteo_hardware/CinteoHardware" />
-    <xacro:base_control mode="${mode}" base_name="${base_name}" />
+    <!-- simulation plugins -->
+    <xacro:if value="${mode == 'simulation_gazebo'}">
+      <xacro:property
+        name="hardware_plugin"
+        value="romea_mobile_base_gazebo/GazeboSystemInterface" />
+    </xacro:if>
+    <xacro:if value="${mode == 'simulation_gazebo_classic'}">
+      <xacro:property name="hardware_plugin"
+        value="romea_mobile_base_gazebo/GazeboSystemInterface1FAS2RWD" />
+    </xacro:if>
+    <xacro:if value="${'4dv' in mode or 'isaac' in mode}">
+      <xacro:property
+        name="hardware_plugin"
+        value="romea_mobile_base_simulation/GenericSimulationSystemInterface" />
+    </xacro:if>
+    <xacro:if value="${mode ==  'live'}">
+      <xacro:property name="hardware_plugin"
+          value="cinteo_hardware/CinteoHardware" />
+    </xacro:if>
+    <xacro:base_control
+      mode="${mode}"
+      base_name="${base_name}"
+      hardware_plugin="${hardware_plugin}" />
   </xacro:macro>
 </robot>
