Commit message: refactoring of some yaml and xacro files
Signed-off-by: jean.laneurit <jean.laneurit@inrae.fr>

File: cinteo_description/urdf/cinteo.xacro (robot description, xacro)
@@ -116,5 +116,6 @@
          </visual>
          <!-- visual front steering -->
-         <box size="${front_wheel_steering_link_xz} ${front_wheel_steering_link_y} ${front_wheel_steering_link_xz}" />
+         <box
+            size="${front_wheel_steering_link_xz} ${front_wheel_steering_link_y} ${front_wheel_steering_link_xz}" />
          <!-- visual front wheel -->
          <cylinder length="${front_wheel_width}" radius="${front_wheel_radius}" />

Commit message: fix steering link mass for simulation

File: cinteo_description/urdf/cinteo.xacro (robot description, xacro)
@@ -106,6 +106,6 @@
       <xacro:property name="maximal_wheel_speed"
          value="${props['rear_wheels_speed_control']['command']['maximal_speed']}" />
-      <xacro:property name="front_wheel_mass" value="5" />
-      <xacro:property name="rear_wheel_mass" value="5" />
+      <xacro:property name="front_wheel_mass" value="10" />
+      <xacro:property name="rear_wheel_mass" value="10" />
       <!-- Steering Properties -->
       <xacro:property name="maximal_axle_steering_angle"
@@ -121,5 +121,5 @@
       <xacro:property name="front_axle_steering_link_y" value="0.05" />
       <xacro:property name="front_axle_steering_link_z" value="0.05" />
-      <xacro:property name="front_wheel_steering_link_mass" value="1" />
+      <xacro:property name="front_wheel_steering_link_mass" value="20" />
       <xacro:property name="front_wheel_steering_link_y" value="${front_hub_carrier_offset}" />
       <xacro:property name="front_wheel_steering_link_xz" value="0.1" />
