Commit message: refactoring
Signed-off-by: Jean Laneurit <jean.laneurit@inrae.fr>

File: cinteo_description/urdf/cinteo.simulation.xacro (robot description, xacro)
@@ -4,5 +4,5 @@
     params="mode ros_prefix base_name controller_manager_config_yaml_file">
     <xacro:if value="${'simulation' in mode}">
-      <xacro:if value="${'gazebo' in  mode}">
+      <xacro:if value="${'gazebo_classic' in  mode}">
         <gazebo>
           <plugin filename="libgazebo_ros2_control.so" name="gazebo_ros2_control">
@@ -17,4 +17,18 @@
         </gazebo>
       </xacro:if>
+      <xacro:if value="${'gazebo_classic' not in  mode}">
+        <gazebo>
+          <plugin filename="gz_ros2_control-system"
+            name="gz_ros2_control::GazeboSimROS2ControlPlugin">
+            <robot_param>robot_description</robot_param>
+            <robot_param_node>ros2_control_description</robot_param_node>
+            <parameters>${controller_manager_config_yaml_file}</parameters>
+            <!-- <hold_joints>true</hold_joints> -->
+            <ros>
+              <namespace>${ros_prefix}${base_name}</namespace>
+            </ros>
+          </plugin>
+        </gazebo>
+      </xacro:if>
     </xacro:if>
   </xacro:macro>

File: cinteo_description/urdf/visual/arms.xacro (robot description, xacro)
@@ -13,10 +13,14 @@
     </xacro:macro>
     <xacro:macro name="front_left_arm_visual">
+        <!-- <xacro:front_arm_visual
+            mesh_filename="package://cinteo_description/meshes/left_wheel_arm.stl" /> -->
         <xacro:front_arm_visual
-            mesh_filename="package://cinteo_description/meshes/left_wheel_arm.stl" />
+            mesh_filename="file://$(find cinteo_description)/meshes/left_wheel_arm.stl" />
     </xacro:macro>
     <xacro:macro name="front_right_arm_visual">
+        <!-- <xacro:front_arm_visual
+            mesh_filename="package://cinteo_description/meshes/right_wheel_arm.stl" /> -->
         <xacro:front_arm_visual
-            mesh_filename="package://cinteo_description/meshes/right_wheel_arm.stl" />
+            mesh_filename="file://$(find cinteo_description)/meshes/right_wheel_arm.stl" />
     </xacro:macro>
 </robot>

File: cinteo_description/urdf/visual/bridge.xacro (robot description, xacro)
@@ -6,5 +6,7 @@
                 <origin xyz="-0.00 0.0 -0.06" rpy="0 0 0" />
                 <geometry>
-                    <mesh filename="package://cinteo_description/meshes/front_bridge.stl"
+                    <!-- <mesh filename="package://cinteo_description/meshes/front_bridge.stl"
+                        scale="0.001 0.001 0.001" /> -->
+                    <mesh filename="file://$(find cinteo_description)/meshes/front_bridge.stl"
                         scale="0.001 0.001 0.001" />
                 </geometry>

File: cinteo_description/urdf/visual/chassis.xacro (robot description, xacro)
@@ -5,5 +5,7 @@
             <origin xyz="0 0 ${chassis_height-0.1}" rpy="0 0 0" />
             <geometry>
-                <mesh filename="package://cinteo_description/meshes/chasis_cinteo.stl"
+                <!-- <mesh filename="package://cinteo_description/meshes/chasis_cinteo.stl"
+                    scale="0.001 0.001 0.001" /> -->
+                <mesh filename="file://$(find cinteo_description)/meshes/chasis_cinteo.stl"
                     scale="0.001 0.001 0.001" />
             </geometry>

File: cinteo_description/urdf/visual/wheels.xacro (robot description, xacro)
@@ -13,6 +13,8 @@
     </xacro:macro>
     <xacro:macro name="rear_wheel_visual">
+        <!-- <xacro:wheel_visual
+            mesh_filename="package://cinteo_description/meshes/rear_wheel.stl" /> -->
         <xacro:wheel_visual
-            mesh_filename="package://cinteo_description/meshes/rear_wheel.stl" />
+            mesh_filename="file://$(find cinteo_description)/meshes/rear_wheel.stl" />
     </xacro:macro>
     <xacro:macro name="rear_left_wheel_visual">
@@ -23,6 +25,8 @@
     </xacro:macro>
     <xacro:macro name="front_wheel_visual">
+        <!-- <xacro:wheel_visual
+            mesh_filename="package://cinteo_description/meshes/front_wheel.stl" /> -->
         <xacro:wheel_visual
-            mesh_filename="package://cinteo_description/meshes/front_wheel.stl" />
+            mesh_filename="file://$(find cinteo_description)/meshes/front_wheel.stl" />
     </xacro:macro>
     <xacro:macro name="front_left_wheel_visual">
